File: VNH2SP30e.brd (EAGLE design)
At the start: 64.2 x 40.7 mm, 17 parts, among them Q1 MOSFET-NCHANNELFDD8580

Commit message: Add files via upload
Parts:
- added LED1, LED2: (no value), led:CHIPLED_1206
- added R10, R11: 1K, SparkFun:1206
- C1: value (none) -> 560uF
- C2: value (none) -> 33nF
- R1, R2, R3, R5, R7: value (none) -> 1K
- R4: value (none) -> 100k
- R6: value (none) -> 4.7K
- R8: value (none) -> 10K
- R9: value (none) -> 1.5K
- moved R4 0.20 mm to (51.0, 3.15)
Connections:
- removed net N$1: U$1.15, U$1.16, U$1.21, U$1.SLUG2, X1.2
- removed net N$14: U$1.1, U$1.25, U$1.30, U$1.SLUG3, X1.1
- new net N$32: LED2.A, R11.1
- new net N$34: LED1.A, R10.1
- new net OUTA: R11.2, U$1.1, U$1.25, U$1.30, U$1.SLUG3, X1.1
- new net OUTB: R10.2, U$1.15, U$1.16, U$1.21, U$1.SLUG2, X1.2
- net GND: now also LED1.C, LED2.C
Routing:
- net OUTA: track 0.00 -> 85.0 mm, vias 0 -> 1
- net OUTB: track 0.00 -> 71.6 mm
- net N$14: track 68.5 -> 0.00 mm
- net N$1: track 66.1 -> 0.00 mm
- net VCC: track 111.5 -> 108.7 mm
Other:
- board size 64.2 x 40.7 mm -> 64.2 x 40.3 mm
