File: VNH2SP30e.sch (EAGLE design)
At the start: 17 parts, among them Q1 MOSFET-NCHANNELFDD8580

Commit message: Add files via upload
Parts:
- added LED1, LED2: (no value), led:LEDCHIPLED_1206
- added R10, R11: 1K, SparkFun:RESISTOR1206
- C1: value (none) -> 560uF
- C2: value (none) -> 33nF
- R1, R2, R3, R5, R7: value (none) -> 1K
- R4: value (none) -> 100k
- R6: value (none) -> 4.7K
- R8: value (none) -> 10K
- R9: value (none) -> 1.5K
Connections:
- removed net N$1: U$1.OUTB@15, U$1.OUTB@16, U$1.OUTB@21, U$1.OUTB@SLUG2, X1-2.SK
- removed net N$14: U$1.OUTA@1, U$1.OUTA@25, U$1.OUTA@30, U$1.OUTA@SLUG3, X1-1.SK
- new net N$32: LED2.A, R11.1
- new net N$34: LED1.A, R10.1
- new net OUTA: R11.2, U$1.OUTA@1, U$1.OUTA@25, U$1.OUTA@30, U$1.OUTA@SLUG3, X1-1.SK
- new net OUTB: R10.2, U$1.OUTB@15, U$1.OUTB@16, U$1.OUTB@21, U$1.OUTB@SLUG2, X1-2.SK
- net GND: now also LED1.C, LED2.C
Changed lines of the file:
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@@
 <part name="P+2" library="supply1" deviceset="+5V" device=""/>
 <part name="GND1" library="supply1" deviceset="GND" device=""/>
-<part name="R1" library="SparkFun" deviceset="RESISTOR" device="1206"/>
-<part name="R2" library="SparkFun" deviceset="RESISTOR" device="1206"/>
-<part name="R3" library="SparkFun" deviceset="RESISTOR" device="1206"/>
-<part name="C1" library="SparkFun" deviceset="CAP_POL" device="G"/>
+<part name="R1" library="SparkFun" deviceset="RESISTOR" device="1206" value="1K"/>
+<part name="R2" library="SparkFun" deviceset="RESISTOR" device="1206" value="1K"/>
+<part name="R3" library="SparkFun" deviceset="RESISTOR" device="1206" value="1K"/>
+<part name="C1" library="SparkFun" deviceset="CAP_POL" device="G" value="560uF"/>
 <part name="P+1" library="SparkFun" deviceset="VCC" device=""/>
 <part name="P+3" library="SparkFun" deviceset="VCC" device=""/>
 <part name="GND2" library="supply1" deviceset="GND" device=""/>
 <part name="P+4" library="SparkFun" deviceset="VCC" device=""/>
-<part name="R4" library="SparkFun" deviceset="RESISTOR" device="1206"/>
+<part name="R4" library="SparkFun" deviceset="RESISTOR" device="1206" value="100k"/>
 <part name="U$2" library="SparkFun" deviceset="DIODE-ZENER" device="SMB" value="DIODE-ZENERSMB"/>
-<part name="R5" library="SparkFun" deviceset="RESISTOR" device="1206"/>
+<part name="R5" library="SparkFun" deviceset="RESISTOR" device="1206" value="1K"/>
 <part name="GND3" library="supply1" deviceset="GND" device=""/>
-<part name="R6" library="SparkFun" deviceset="RESISTOR" device="1206"/>
-<part name="R7" library="SparkFun" deviceset="RESISTOR" device="1206"/>
-<part name="R8" library="SparkFun" deviceset="RESISTOR" device="1206"/>
-<part name="R9" library="SparkFun" deviceset="RESISTOR" device="1206"/>
+<part name="R6" library="SparkFun" deviceset="RESISTOR" device="1206" value="4.7K"/>
+<part name="R7" library="SparkFun" deviceset="RESISTOR" device="1206" value="1K"/>
+<part name="R8" library="SparkFun" deviceset="RESISTOR" device="1206" value="10K"/>
+<part name="R9" library="SparkFun" deviceset="RESISTOR" device="1206" value="1.5K"/>
 <part name="GND4" library="supply1" deviceset="GND" device=""/>
-<part name="C2" library="SparkFun" deviceset="CAP" device="1206"/>
+<part name="C2" library="SparkFun" deviceset="CAP" device="1206" value="33nF"/>
 <part name="GND5" library="supply1" deviceset="GND" device=""/>
 <part name="X1" library="con-phoenix-500" deviceset="MSTBV2" device=""/>
@@
 <part name="GND6" library="supply1" deviceset="GND" device=""/>
 <part name="JP1" library="pinhead" deviceset="PINHD-1X7" device=""/>
+<part name="LED1" library="led" deviceset="LED" device="CHIPLED_1206"/>
+<part name="R10" library="SparkFun" deviceset="RESISTOR" device="1206" value="1K"/>
+<part name="LED2" library="led" deviceset="LED" device="CHIPLED_1206"/>
+<part name="R11" library="SparkFun" deviceset="RESISTOR" device="1206" value="1K"/>
+<part name="GND7" library="supply1" deviceset="GND" device=""/>
 </parts>
 <sheets>
@@
 <instance part="GND6" gate="1" x="12.7" y="81.28" rot="R180"/>
 <instance part="JP1" gate="A" x="7.62" y="40.64" rot="R180"/>
+<instance part="LED1" gate="G$1" x="134.62" y="0" rot="R90"/>
+<instance part="R10" gate="G$1" x="124.46" y="0" rot="R180"/>
+<instance part="LED2" gate="G$1" x="134.62" y="-10.16" rot="R90"/>
+<instance part="R11" gate="G$1" x="124.46" y="-10.16" rot="R180"/>
+<instance part="GND7" gate="1" x="142.24" y="-15.24"/>
 </instances>
 <busses>
@@
 <pinref part="JP1" gate="A" pin="1"/>
 <wire x1="10.16" y1="33.02" x2="17.78" y2="33.02" width="0.1524" layer="91"/>
+</segment>
+<segment>
+<pinref part="LED1" gate="G$1" pin="C"/>
+<wire x1="139.7" y1="0" x2="142.24" y2="0" width="0.1524" layer="91"/>
+<wire x1="142.24" y1="0" x2="142.24" y2="-10.16" width="0.1524" layer="91"/>
+<pinref part="LED2" gate="G$1" pin="C"/>
+<wire x1="142.24" y1="-10.16" x2="139.7" y2="-10.16" width="0.1524" layer="91"/>
+<pinref part="GND7" gate="1" pin="GND"/>
+<wire x1="142.24" y1="-12.7" x2="142.24" y2="-10.16" width="0.1524" layer="91"/>
 </segment>
 </net>
@@
 </segment>
 </net>
-<net name="N$14" class="0">
+<net name="N$11" class="0">
+<segment>
+<pinref part="U$1" gate="G$1" pin="CS"/>
+<pinref part="R8" gate="G$1" pin="1"/>
+<wire x1="91.44" y1="27.94" x2="93.98" y2="27.94" width="0.1524" layer="91"/>
+<pinref part="R9" gate="G$1" pin="2"/>
+<wire x1="93.98" y1="27.94" x2="96.52" y2="27.94" width="0.1524" layer="91"/>
+<wire x1="93.98" y1="25.4" x2="93.98" y2="27.94" width="0.1524" layer="91"/>
+<junction x="93.98" y="27.94"/>
+</segment>
+</net>
+<net name="CS" class="0">
+<segment>
+<pinref part="R8" gate="G$1" pin="2"/>
+<wire x1="106.68" y1="27.94" x2="109.22" y2="27.94" width="0.1524" layer="91"/>
+<pinref part="C2" gate="G$1" pin="1"/>
+<wire x1="109.22" y1="27.94" x2="111.76" y2="27.94" width="0.1524" layer="91"/>
+<wire x1="109.22" y1="25.4" x2="109.22" y2="27.94" width="0.1524" layer="91"/>
+<junction x="109.22" y="27.94"/>
+</segment>
+<segment>
+<wire x1="10.16" y1="35.56" x2="17.78" y2="35.56" width="0.1524" layer="91"/>
+<pinref part="JP1" gate="A" pin="2"/>
+</segment>
+</net>
+<net name="N$34" class="0">
+<segment>
+<pinref part="LED1" gate="G$1" pin="A"/>
+<wire x1="129.54" y1="0" x2="132.08" y2="0" width="0.1524" layer="91"/>
+<pinref part="R10" gate="G$1" pin="1"/>
+</segment>
+</net>
+<net name="N$32" class="0">
+<segment>
+<pinref part="LED2" gate="G$1" pin="A"/>
+<wire x1="129.54" y1="-10.16" x2="132.08" y2="-10.16" width="0.1524" layer="91"/>
+<pinref part="R11" gate="G$1" pin="1"/>
+</segment>
+</net>
+<net name="OUTB" class="0">
+<segment>
+<pinref part="R10" gate="G$1" pin="2"/>
+<wire x1="119.38" y1="0" x2="116.84" y2="0" width="0.1524" layer="91"/>
+</segment>
+<segment>
+<pinref part="U$1" gate="G$1" pin="OUTB@15"/>
+<wire x1="91.44" y1="33.02" x2="93.98" y2="33.02" width="0.1524" layer="91"/>
+<wire x1="93.98" y1="33.02" x2="93.98" y2="35.56" width="0.1524" layer="91"/>
+<pinref part="U$1" gate="G$1" pin="OUTB@16"/>
+<wire x1="93.98" y1="35.56" x2="93.98" y2="38.1" width="0.1524" layer="91"/>
+<wire x1="93.98" y1="38.1" x2="93.98" y2="40.64" width="0.1524" layer="91"/>
+<wire x1="91.44" y1="35.56" x2="93.98" y2="35.56" width="0.1524" layer="91"/>
+<pinref part="U$1" gate="G$1" pin="OUTB@21"/>
+<wire x1="91.44" y1="38.1" x2="93.98" y2="38.1" width="0.1524" layer="91"/>
+<junction x="93.98" y="35.56"/>
+<junction x="93.98" y="38.1"/>
+<pinref part="U$1" gate="G$1" pin="OUTB@SLUG2"/>
+<wire x1="91.44" y1="40.64" x2="93.98" y2="40.64" width="0.1524" layer="91"/>
+<junction x="93.98" y="40.64"/>
+<wire x1="93.98" y1="40.64" x2="114.3" y2="40.64" width="0.1524" layer="91"/>
+<pinref part="X1" gate="-2" pin="SK"/>
+<wire x1="114.3" y1="45.72" x2="114.3" y2="40.64" width="0.1524" layer="91"/>
+</segment>
+</net>
+<net name="OUTA" class="0">
+<segment>
+<pinref part="R11" gate="G$1" pin="2"/>
+<wire x1="119.38" y1="-10.16" x2="116.84" y2="-10.16" width="0.1524" layer="91"/>
+</segment>
 <segment>
 <pinref part="U$1" gate="G$1" pin="OUTA@SLUG3"/>
@@
 </segment>
 </net>
-<net name="N$1" class="0">
-<segment>
-<pinref part="U$1" gate="G$1" pin="OUTB@15"/>
-<wire x1="91.44" y1="33.02" x2="93.98" y2="33.02" width="0.1524" layer="91"/>
-<wire x1="93.98" y1="33.02" x2="93.98" y2="35.56" width="0.1524" layer="91"/>
-<pinref part="U$1" gate="G$1" pin="OUTB@16"/>
-<wire x1="93.98" y1="35.56" x2="93.98" y2="38.1" width="0.1524" layer="91"/>
-<wire x1="93.98" y1="38.1" x2="93.98" y2="40.64" width="0.1524" layer="91"/>
-<wire x1="91.44" y1="35.56" x2="93.98" y2="35.56" width="0.1524" layer="91"/>
-<pinref part="U$1" gate="G$1" pin="OUTB@21"/>
-<wire x1="91.44" y1="38.1" x2="93.98" y2="38.1" width="0.1524" layer="91"/>
-<junction x="93.98" y="35.56"/>
-<junction x="93.98" y="38.1"/>
-<pinref part="U$1" gate="G$1" pin="OUTB@SLUG2"/>
-<wire x1="91.44" y1="40.64" x2="93.98" y2="40.64" width="0.1524" layer="91"/>
-<junction x="93.98" y="40.64"/>
-<wire x1="93.98" y1="40.64" x2="114.3" y2="40.64" width="0.1524" layer="91"/>
-<pinref part="X1" gate="-2" pin="SK"/>
-<wire x1="114.3" y1="45.72" x2="114.3" y2="40.64" width="0.1524" layer="91"/>
-</segment>
-</net>
-<net name="N$11" class="0">
-<segment>
-<pinref part="U$1" gate="G$1" pin="CS"/>
-<pinref part="R8" gate="G$1" pin="1"/>
-<wire x1="91.44" y1="27.94" x2="93.98" y2="27.94" width="0.1524" layer="91"/>
-<pinref part="R9" gate="G$1" pin="2"/>
-<wire x1="93.98" y1="27.94" x2="96.52" y2="27.94" width="0.1524" layer="91"/>
-<wire x1="93.98" y1="25.4" x2="93.98" y2="27.94" width="0.1524" layer="91"/>
-<junction x="93.98" y="27.94"/>
-</segment>
-</net>
-<net name="CS" class="0">
-<segment>
-<pinref part="R8" gate="G$1" pin="2"/>
-<wire x1="106.68" y1="27.94" x2="109.22" y2="27.94" width="0.1524" layer="91"/>
-<pinref part="C2" gate="G$1" pin="1"/>
-<wire x1="109.22" y1="27.94" x2="111.76" y2="27.94" width="0.1524" layer="91"/>
-<wire x1="109.22" y1="25.4" x2="109.22" y2="27.94" width="0.1524" layer="91"/>
-<junction x="109.22" y="27.94"/>
-</segment>
-<segment>
-<wire x1="10.16" y1="35.56" x2="17.78" y2="35.56" width="0.1524" layer="91"/>
-<pinref part="JP1" gate="A" pin="2"/>
-</segment>
-</net>
